File: KiCAD/Mainboard/IM350/IM350/IM350- Single.kicad_pcb (KiCad board)
At the start: 2 copper layers, 31 x 47.5 mm, 13 parts, among them J1 USB_B_Micro_Power, J2 Conn_02x03_Odd_Even, Q1 BC547, SW1 SW_Push, U1 AMS1117-3.3, U2 ESP-12F

Commit message: Update
Parts:
- removed U1: AMS1117-3.3, Package_TO_SOT_SMD:SOT-223-3_TabPin2
- added IC1: ME6211C33M5G, ErichCollection:SOT95P282X145-5N, F.Cu at (58.0, 78.0)
- C1, C2: value 22uF -> C; footprint Capacitor_SMD:C_1206_3216Metric_Pad1.33x1.80mm_HandSolder -> Capacitor_SMD:C_0805_2012Metric_Pad1.18x1.45mm_HandSolder
- moved C2 4.47 mm to (56.5, 73.0), turned to 90 degrees
- moved C1 3.16 mm to (59.5, 73.0), turned to 90 degrees
Connections:
- C1 pad 1: GND -> +5V
- C1 pad 2: +5V -> GND
Routing:
- net +3V3: track 90.4 -> 52.1 mm, vias 1 -> 0
- net GND: track 116.2 -> 98.7 mm
- net +5V: track 14.7 -> 13.6 mm
