File: KiCAD/Mainboard/IM350/IM350/IM350.kicad_pcb (KiCad board)
At the start: 2 copper layers, 95 x 96 mm, 78 parts, among them J1 USB_B_Micro_Power, J2 Conn_02x03_Odd_Even, Q1 BC547, SW1 SW_Push, U1 AMS1117-3.3, U2 ESP-12F

Commit message: Update
Parts:
- removed the C1 at (120.5, 72.0)
- removed the C1 at (120.5, 120.5)
- removed the C1 at (88.5, 72.0)
- removed the C1 at (88.5, 120.5)
- removed the C1 at (56.5, 120.5)
- removed the C2 at (122.5, 69.0)
- removed the C2 at (122.5, 117.5)
- removed the C2 at (90.5, 69.0)
- removed the C2 at (90.5, 117.5)
- removed the C2 at (58.5, 117.5)
- removed the G*** at (122.5, 113.0)
- removed the G*** at (58.5, 113.0)
- removed the G*** at (130.0, 113.5)
- removed the G*** at (130.0, 65.0)
- removed the G*** at (122.5, 64.5)
- removed the G*** at (90.5, 113.0)
- removed the G*** at (98.0, 113.5)
- removed the G*** at (98.0, 65.0)
- removed the G*** at (90.5, 64.5)
- removed the G*** at (66.0, 113.5)
- removed J1 (x6): USB_B_Micro_Power, SHRDZM:USB_Micro-B_Power
- removed the J2 at (70.0, 92.5)
- removed the J2 at (102.0, 92.5)
- removed the J2 at (102.0, 44.0)
- removed the J2 at (134.0, 44.0)
- removed the J2 at (134.0, 92.5)
- removed the Q1 at (130.5, 47.5)
- removed the Q1 at (130.5, 96.0)
- removed the Q1 at (98.5, 47.5)
- removed the Q1 at (98.5, 96.0)
- removed the Q1 at (66.5, 96.0)
- removed the R1 at (134.5, 96.0)
- removed the R1 at (134.5, 47.5)
- removed the R1 at (102.5, 96.0)
- removed the R1 at (102.5, 47.5)
- removed the R1 at (70.5, 96.0)
- removed the R2 at (139.0, 96.0)
- removed the R2 at (139.0, 47.5)
- removed the R2 at (107.0, 96.0)
- removed the R2 at (107.0, 47.5)
- removed the R2 at (75.0, 96.0)
- removed the R3 at (145.0, 119.5)
- removed the R3 at (145.0, 71.0)
- removed the R3 at (113.0, 119.5)
- removed the R3 at (113.0, 71.0)
- removed the R3 at (81.0, 119.5)
- removed the SW1 at (137.5, 124.5)
- removed the SW1 at (137.5, 76.0)
- removed the SW1 at (105.5, 124.5)
- removed the SW1 at (105.5, 76.0)
- removed the SW1 at (73.5, 124.5)
- removed the U1 at (121.5, 126.5)
- removed the U1 at (121.5, 78.0)
- removed the U1 at (89.5, 126.5)
- removed the U1 at (89.5, 78.0)
- removed the U1 at (57.5, 126.5)
- removed the U2 at (134.5, 61.0)
- removed the U2 at (134.5, 109.5)
- removed the U2 at (102.5, 109.5)
- removed the U2 at (102.5, 61.0)
- removed the U2 at (70.5, 109.5)
Routing:
- net GND: track 697.0 -> 116.2 mm
- net +3V3: track 542.5 -> 90.4 mm, vias 6 -> 1
- net Net-(Q1-Pad1): track 193.1 -> 32.2 mm
- net Net-(J2-Pad2): track 183.4 -> 30.6 mm
- net Net-(J2-Pad5): track 173.8 -> 29.0 mm
- net Net-(SW1-Pad1): track 135.3 -> 22.6 mm
- net +5V: track 88.2 -> 14.7 mm
- net Net-(R3-Pad2): track 18.6 -> 3.11 mm
Other:
- board size 95 x 96 mm -> 31 x 47.5 mm
