File: KiCAD/Mainboard/DOORSENSOR_Enhanced/DOORSENSOR_Enhanced/DOORSENSOR_Enhanced_AutoRoute.kicad_pcb (KiCad board)
At the start: 2 copper layers, 70 x 20 mm, 13 parts, among them J1 Power, Q1 2N2222, Q2 NDP6020P, SW1 Trigger, SW2 Pairing, SW3 Open/Close, U1 ESP-12F

Commit message: Update
Connections:
- U1 pad 4: Net-(U1-Pad4) -> Net-(U1-Pad1)
Routing:
- net Net-(U1-Pad1): track 0.00 -> 9.15 mm
Changed lines of the file:
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@@
     (thickness 1.6)
     (drawings 8)
-    (tracks 72)
+    (tracks 75)
     (zones 0)
     (modules 13)
-    (nets 25)
+    (nets 24)
   )
   (page A4)
@@
   (net 8 "Net-(U1-Pad1)")
   (net 9 "Net-(U1-Pad2)")
-  (net 10 "Net-(U1-Pad4)")
-  (net 11 "Net-(U1-Pad6)")
-  (net 12 "Net-(U1-Pad9)")
-  (net 13 "Net-(U1-Pad10)")
-  (net 14 "Net-(U1-Pad11)")
-  (net 15 "Net-(U1-Pad12)")
-  (net 16 "Net-(U1-Pad13)")
-  (net 17 "Net-(U1-Pad14)")
-  (net 18 "Net-(U1-Pad17)")
-  (net 19 "Net-(U1-Pad18)")
-  (net 20 "Net-(U1-Pad19)")
-  (net 21 "Net-(U1-Pad21)")
-  (net 22 "Net-(U1-Pad22)")
-  (net 23 "Net-(Q1-Pad2)")
-  (net 24 "Net-(Q1-Pad3)")
+  (net 10 "Net-(U1-Pad6)")
+  (net 11 "Net-(U1-Pad9)")
+  (net 12 "Net-(U1-Pad10)")
+  (net 13 "Net-(U1-Pad11)")
+  (net 14 "Net-(U1-Pad12)")
+  (net 15 "Net-(U1-Pad13)")
+  (net 16 "Net-(U1-Pad14)")
+  (net 17 "Net-(U1-Pad17)")
+  (net 18 "Net-(U1-Pad18)")
+  (net 19 "Net-(U1-Pad19)")
+  (net 20 "Net-(U1-Pad21)")
+  (net 21 "Net-(U1-Pad22)")
+  (net 22 "Net-(Q1-Pad2)")
+  (net 23 "Net-(Q1-Pad3)")
   (net_class Default "This is the default net class."
     (clearance 0.2)
@@
     (add_net "Net-(U1-Pad21)")
     (add_net "Net-(U1-Pad22)")
-    (add_net "Net-(U1-Pad4)")
     (add_net "Net-(U1-Pad6)")
     (add_net "Net-(U1-Pad9)")
@@
       (net 2 GND))
     (pad 3 thru_hole oval (at 2.54 0 90) (size 1.05 1.5) (drill 0.75) (layers *.Cu *.Mask)
-      (net 24 "Net-(Q1-Pad3)"))
+      (net 23 "Net-(Q1-Pad3)"))
     (pad 2 thru_hole oval (at 1.27 0 90) (size 1.05 1.5) (drill 0.75) (layers *.Cu *.Mask)
-      (net 23 "Net-(Q1-Pad2)"))
+      (net 22 "Net-(Q1-Pad2)"))
     (model ${KISYS3DMOD}/Package_TO_SOT_THT.3dshapes/TO-92_Inline.wrl
       (at (xyz 0 0 0))
@@
       (net 5 "Net-(Q2-Pad2)"))
     (pad 1 thru_hole rect (at 0 0 270) (size 1.905 2) (drill 1.1) (layers *.Cu *.Mask)
-      (net 24 "Net-(Q1-Pad3)"))
+      (net 23 "Net-(Q1-Pad3)"))
     (pad "" np_thru_hole oval (at 2.54 -16.66 270) (size 3.5 3.5) (drill 3.5) (layers *.Cu *.Mask))
     (model ${KISYS3DMOD}/Package_TO_SOT_THT.3dshapes/TO-220-3_Horizontal_TabDown.wrl
@@
     )
     (pad 1 thru_hole circle (at 0 0 90) (size 1.4 1.4) (drill 0.7) (layers *.Cu *.Mask)
-      (net 23 "Net-(Q1-Pad2)"))
+      (net 22 "Net-(Q1-Pad2)"))
     (pad 2 thru_hole oval (at 2.54 0 90) (size 1.4 1.4) (drill 0.7) (layers *.Cu *.Mask)
       (net 1 "Net-(C1-Pad1)"))
@@
     )
     (pad 2 thru_hole oval (at 2.54 0 90) (size 1.4 1.4) (drill 0.7) (layers *.Cu *.Mask)
-      (net 24 "Net-(Q1-Pad3)"))
+      (net 23 "Net-(Q1-Pad3)"))
     (pad 1 thru_hole circle (at 0 0 90) (size 1.4 1.4) (drill 0.7) (layers *.Cu *.Mask)
       (net 4 +3V3))
@@
       (net 5 "Net-(Q2-Pad2)"))
     (pad 4 smd rect (at -7.6 2.5 90) (size 2.5 1) (layers F.Cu F.Paste F.Mask)
-      (net 10 "Net-(U1-Pad4)"))
+      (net 8 "Net-(U1-Pad1)"))
     (pad 5 smd rect (at -7.6 4.5 90) (size 2.5 1) (layers F.Cu F.Paste F.Mask)
       (net 3 "Net-(D1-Pad2)"))
     (pad 6 smd rect (at -7.6 6.5 90) (size 2.5 1) (layers F.Cu F.Paste F.Mask)
-      (net 11 "Net-(U1-Pad6)"))
+      (net 10 "Net-(U1-Pad6)"))
     (pad 7 smd rect (at -7.6 8.5 90) (size 2.5 1) (layers F.Cu F.Paste F.Mask)
       (net 6 "Net-(SW2-Pad1)"))
@@
       (net 5 "Net-(Q2-Pad2)"))
     (pad 9 smd rect (at -5 12 90) (size 1 1.8) (layers F.Cu F.Paste F.Mask)
-      (net 12 "Net-(U1-Pad9)"))
+      (net 11 "Net-(U1-Pad9)"))
     (pad 10 smd rect (at -3 12 90) (size 1 1.8) (layers F.Cu F.Paste F.Mask)
-      (net 13 "Net-(U1-Pad10)"))
+      (net 12 "Net-(U1-Pad10)"))
     (pad 11 smd rect (at -1 12 90) (size 1 1.8) (layers F.Cu F.Paste F.Mask)
-      (net 14 "Net-(U1-Pad11)"))
+      (net 13 "Net-(U1-Pad11)"))
     (pad 12 smd rect (at 1 12 90) (size 1 1.8) (layers F.Cu F.Paste F.Mask)
-      (net 15 "Net-(U1-Pad12)"))
+      (net 14 "Net-(U1-Pad12)"))
     (pad 13 smd rect (at 3 12 90) (size 1 1.8) (layers F.Cu F.Paste F.Mask)
-      (net 16 "Net-(U1-Pad13)"))
+      (net 15 "Net-(U1-Pad13)"))
     (pad 14 smd rect (at 5 12 90) (size 1 1.8) (layers F.Cu F.Paste F.Mask)
-      (net 17 "Net-(U1-Pad14)"))
+      (net 16 "Net-(U1-Pad14)"))
     (pad 15 smd rect (at 7.6 10.5 90) (size 2.5 1) (layers F.Cu F.Paste F.Mask)
       (net 2 GND))
@@
       (net 2 GND))
     (pad 17 smd rect (at 7.6 6.5 90) (size 2.5 1) (layers F.Cu F.Paste F.Mask)
-      (net 18 "Net-(U1-Pad17)"))
+      (net 17 "Net-(U1-Pad17)"))
     (pad 18 smd rect (at 7.6 4.5 90) (size 2.5 1) (layers F.Cu F.Paste F.Mask)
-      (net 19 "Net-(U1-Pad18)"))
+      (net 18 "Net-(U1-Pad18)"))
     (pad 19 smd rect (at 7.6 2.5 90) (size 2.5 1) (layers F.Cu F.Paste F.Mask)
-      (net 20 "Net-(U1-Pad19)"))
+      (net 19 "Net-(U1-Pad19)"))
     (pad 20 smd rect (at 7.6 0.5 90) (size 2.5 1) (layers F.Cu F.Paste F.Mask)
       (net 7 "Net-(SW3-Pad1)"))
     (pad 21 smd rect (at 7.6 -1.5 90) (size 2.5 1) (layers F.Cu F.Paste F.Mask)
-      (net 21 "Net-(U1-Pad21)"))
+      (net 20 "Net-(U1-Pad21)"))
     (pad 22 smd rect (at 7.6 -3.5 90) (size 2.5 1) (layers F.Cu F.Paste F.Mask)
-      (net 22 "Net-(U1-Pad22)"))
+      (net 21 "Net-(U1-Pad22)"))
     (model ${KISYS3DMOD}/RF_Module.3dshapes/ESP-12E.wrl
       (at (xyz 0 0 0))
@@
   (segment (start 76.8807 49.959) (end 85 58.0783) (width 0.25) (layer F.Cu) (net 7))
   (segment (start 85 58.0783) (end 85 61.5) (width 0.25) (layer F.Cu) (net 7))
-  (segment (start 77 47.5) (end 77.77 46.73) (width 0.25) (layer F.Cu) (net 23))
-  (segment (start 77.77 46.73) (end 81.5 46.73) (width 0.25) (layer F.Cu) (net 23))
-  (segment (start 81.5 45.46) (end 82.5753 45.46) (width 0.25) (layer B.Cu) (net 24))
-  (segment (start 77 52.5) (end 78.7604 52.5) (width 0.25) (layer B.Cu) (net 24))
-  (segment (start 78.7604 52.5) (end 82.5753 48.6851) (width 0.25) (layer B.Cu) (net 24))
-  (segment (start 82.5753 48.6851) (end 82.5753 45.46) (width 0.25) (layer B.Cu) (net 24))
-  (segment (start 74.5 56.96) (end 74.5 55) (width 0.25) (layer B.Cu) (net 24))
-  (segment (start 74.5 55) (end 77 52.5) (width 0.25) (layer B.Cu) (net 24))
+  (segment (start 46 60.6) (end 46 59.0247) (width 0.25) (layer F.Cu) (net 8))
+  (segment (start 52 60.6) (end 52 59.0247) (width 0.25) (layer F.Cu) (net 8))
+  (segment (start 52 59.0247) (end 46 59.0247) (width 0.25) (layer F.Cu) (net 8))
+  (segment (start 77 47.5) (end 77.77 46.73) (width 0.25) (layer F.Cu) (net 22))
+  (segment (start 77.77 46.73) (end 81.5 46.73) (width 0.25) (layer F.Cu) (net 22))
+  (segment (start 81.5 45.46) (end 82.5753 45.46) (width 0.25) (layer B.Cu) (net 23))
+  (segment (start 77 52.5) (end 78.7604 52.5) (width 0.25) (layer B.Cu) (net 23))
+  (segment (start 78.7604 52.5) (end 82.5753 48.6851) (width 0.25) (layer B.Cu) (net 23))
+  (segment (start 82.5753 48.6851) (end 82.5753 45.46) (width 0.25) (layer B.Cu) (net 23))
+  (segment (start 74.5 56.96) (end 74.5 55) (width 0.25) (layer B.Cu) (net 23))
+  (segment (start 74.5 55) (end 77 52.5) (width 0.25) (layer B.Cu) (net 23))
 )
