File: KiCAD/Mainboard/DOORSENSOR_Enhanced/DOORSENSOR_Enhanced/DOORSENSOR_Enhanced_Multi.kicad_pcb (KiCad board)
At the start: 2 copper layers, 90 x 100 mm, 151 parts, among them J1 Power, Q1 2N2222, Q2 NDP6020P, SW1 Trigger, SW2 Pairing, SW3 Open/Close, U1 ESP-12F

Commit message: Update
Connections:
- U1 pad 4: Net-(U1-Pad4) -> Net-(U1-Pad1) (x12)
Routing:
- net Net-(U1-Pad1): track 0.00 -> 54.4 mm
Other:
- board text added: "V1.1"
- board text removed: "V1.0"
