File: KiCAD/Mainboard/DOORSENSOR_Enhanced/DOORSENSOR_Enhanced/DOORSENSOR_Enhanced.kicad_pcb (KiCad board)
At the start: 2 copper layers, 70 x 20 mm, 11 parts, among them J1 Power, Q1 2N2222, Q2 NDP6020P, SW1 Trigger, SW2 Pairing, SW3 Open/Close, U1 ESP-12F

Commit message: Update
Parts:
- added G***: LOGO, SHRDZM:SHRDZM 33x11, B.Cu at (54.0, 50.5)
- added G***: LOGO, SHRDZM:SHRDZM Symbol 5x5, F.Cu at (101.0, 59.5)
Other:
- board text added: "V1.0"
- board text added: "www.shrdzm.com"

Commit message: Bootreason added
Connections:
- U1 pad 4: Net-(U1-Pad4) -> Net-(U1-Pad1)
Routing:
- net Net-(U1-Pad1): track 0.00 -> 9.06 mm
Other:
- board text added: "V1.1"
- board text removed: "V1.0"

Commit message: Update
Routing:
- net GND: track 73.8 -> 0.00 mm
- net Net-(SW3-Pad1): track 43.8 -> 0.00 mm, vias 1 -> 0
- net +3V3: track 38.0 -> 0.00 mm
- net Net-(Q2-Pad2): track 35.6 -> 0.00 mm
- net Net-(C1-Pad1): track 23.6 -> 0.00 mm
- net Net-(Q1-Pad3): track 21.8 -> 0.00 mm
- net Net-(SW2-Pad1): track 15.8 -> 0.00 mm
- net Net-(D1-Pad2): track 14.7 -> 0.00 mm
- net Net-(U1-Pad1): track 9.06 -> 0.00 mm
- net Net-(Q1-Pad2): track 4.82 -> 0.00 mm
Other:
- board text added: "V2.0"
- board text removed: "V1.1"
