File: KiCAD/IM350_AM550_5V_SMD/IM350_AM550_5V_SMD.kicad_pcb (KiCad board)
At the start: 2 copper layers, 10 parts, among them J5 USB_B_Micro_Power, J7 RJ12, P3 0R, P4 0R, SW1 Pairing, U1 MCP1700-3302E_SOT23, U2 ESP-12F

Commit message: Update
Other:
- board outline added: 35 x 19 mm

Commit message: Update
Parts:
- moved J5 9.00 mm to (78.5, 39.1)
Other:
- board size 35 x 19 mm -> 43 x 19 mm
Changed lines of the file:
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@@
       (rotate (xyz 0 0 0))
+    )
+    (model C:/Users/erich/Nextcloud/Diverses/KiCAD/model/95501-2661.wrl
+      (offset (xyz 3.2 -17 5.75))
+      (scale (xyz 400 400 400))
+      (rotate (xyz -90 0 0))
     )
   )
@@
   )
   (module SHRDZM:USB_Micro-B_Power (layer B.Cu)
-    (at 69.5 39.25 270)
+    (at 78.5 39.1 270)
     (tags "Micro-USB Power")
     (attr smd)
@@
     )
   )
-  (gr_line (start 38.1 29.8) (end 73.1 29.8) (layer Edge.Cuts) (width 0.05))
+  (gr_line (start 81.1 29.8) (end 81.1 48.8) (layer Edge.Cuts) (width 0.05))
+  (gr_line (start 38.1 29.8) (end 81.1 29.8) (layer Edge.Cuts) (width 0.05))
   (gr_line (start 38.1 48.8) (end 38.1 29.8) (layer Edge.Cuts) (width 0.05))
-  (gr_line (start 73.1 48.8) (end 38.1 48.8) (layer Edge.Cuts) (width 0.05))
-  (gr_line (start 73.1 29.8) (end 73.1 48.8) (layer Edge.Cuts) (width 0.05))
+  (gr_line (start 81.1 48.8) (end 38.1 48.8) (layer Edge.Cuts) (width 0.05))
   (dimension 19 (width 0.15) (layer Dwgs.User)
     (gr_text "19,000 mm" (at 78.9 39.3 270) (layer Dwgs.User)
