File: KiCAD/Mainboard/GatewayMQTT/DOORSENSOR/DOORSENSOR.sch (KiCad schematic (older format))
At the start: 9 parts, among them J4 Power, Q1 IRLZ44N, SW1 Trigger, SW2 Pairing, SW3 Open/Close, U1 ESP-12F

Commit message: Update 3D Models
Connections:
- net GND: now also Q1.3 (S); no longer C2.1, Q1.2 (D), SW2.2, SW3.2, U1.15 (GND), U1.16 (GPIO15)
- net at C1.1, Q1.1 (G), SW1.2: now also R1.1
- new net: C2.1, Q1.2 (D), SW2.2, SW3.2, U1.15 (GND), U1.16 (GPIO15)
Other:
- moved on the sheet: Q1, R1
Changed lines of the file:
@@
 L Transistor_FET:IRLZ44N Q1
 U 1 1 605A127B
-P 2100 3350
-F 0 "Q1" H 2050 3600 50  0000 L CNN
-F 1 "IRLZ44N" H 1850 3500 50  0000 L CNN
-F 2 "Package_TO_SOT_THT:TO-220-3_Horizontal_TabDown" H 2350 3275 50  0001 L CIN
-F 3 "http://www.irf.com/product-info/datasheets/data/irlz44n.pdf" H 2100 3350 50  0001 L CNN
-	1    2100 3350
-	1    0    0    -1
-$EndComp
-$Comp
-L power:GND #PWR06
-U 1 1 605A5E2A
-P 2550 3850
-F 0 "#PWR06" H 2550 3600 50  0001 C CNN
-F 1 "GND" H 2555 3677 50  0000 C CNN
-F 2 "" H 2550 3850 50  0001 C CNN
-F 3 "" H 2550 3850 50  0001 C CNN
-	1    2550 3850
-	1    0    0    -1
-$EndComp
-Wire Wire Line
-	2550 3150 2550 3850
-Wire Wire Line
-	2550 3150 2200 3150
+P 2350 3350
+F 0 "Q1" H 2300 3600 50  0000 L CNN
+F 1 "IRLZ44N" H 2100 3500 50  0000 L CNN
+F 2 "Package_TO_SOT_THT:TO-220-3_Horizontal_TabDown" H 2600 3275 50  0001 L CIN
+F 3 "http://www.irf.com/product-info/datasheets/data/irlz44n.pdf" H 2350 3350 50  0001 L CNN
+	1    2350 3350
+	1    0    0    -1
+$EndComp
 $Comp
 L Switch:SW_Reed SW1
@@
 Wire Wire Line
 	1550 3250 1550 3350
-Wire Wire Line
-	1550 3350 1900 3350
 $Comp
 L power:+3.3V #PWR03
@@
 L Device:R R1
 U 1 1 605B1A6F
-P 2200 3700
-F 0 "R1" H 2270 3746 50  0000 L CNN
-F 1 "R" H 2270 3655 50  0000 L CNN
-F 2 "Resistor_THT:R_Axial_DIN0207_L6.3mm_D2.5mm_P10.16mm_Horizontal" V 2130 3700 50  0001 C CNN
-F 3 "~" H 2200 3700 50  0001 C CNN
-	1    2200 3700
+P 1950 3600
+F 0 "R1" H 2020 3646 50  0000 L CNN
+F 1 "R" H 2020 3555 50  0000 L CNN
+F 2 "Resistor_THT:R_Axial_DIN0207_L6.3mm_D2.5mm_P10.16mm_Horizontal" V 1880 3600 50  0001 C CNN
+F 3 "~" H 1950 3600 50  0001 C CNN
+	1    1950 3600
 	1    0    0    -1
 $EndComp
@@
 L power:GND #PWR05
 U 1 1 605B237C
-P 2200 3850
-F 0 "#PWR05" H 2200 3600 50  0001 C CNN
-F 1 "GND" H 2205 3677 50  0000 C CNN
-F 2 "" H 2200 3850 50  0001 C CNN
-F 3 "" H 2200 3850 50  0001 C CNN
-	1    2200 3850
+P 1950 3850
+F 0 "#PWR05" H 1950 3600 50  0001 C CNN
+F 1 "GND" H 1955 3677 50  0000 C CNN
+F 2 "" H 1950 3850 50  0001 C CNN
+F 3 "" H 1950 3850 50  0001 C CNN
+	1    1950 3850
 	1    0    0    -1
 $EndComp
@@
 Wire Wire Line
 	4650 2450 4900 2450
-$Comp
-L power:GND #PWR08
-U 1 1 6062D75E
-P 4050 3850
-F 0 "#PWR08" H 4050 3600 50  0001 C CNN
-F 1 "GND" H 4055 3677 50  0000 C CNN
-F 2 "" H 4050 3850 50  0001 C CNN
-F 3 "" H 4050 3850 50  0001 C CNN
-	1    4050 3850
-	1    0    0    -1
-$EndComp
 Wire Wire Line
 	4050 3050 4050 3250
@@
 Connection ~ 4050 3250
 Wire Wire Line
-	4050 3250 4050 3850
+	4050 3250 4050 3500
 $Comp
 L Switch:SW_Push SW2
@@
 NoConn ~ 4650 1850
 NoConn ~ 4650 2050
+Wire Wire Line
+	1950 3350 1950 3450
+Wire Wire Line
+	1950 3850 1950 3750
+Wire Wire Line
+	4050 3500 3050 3500
+Wire Wire Line
+	3050 3500 3050 2950
+Wire Wire Line
+	3050 2950 2450 2950
+Wire Wire Line
+	2450 2950 2450 3150
+Wire Wire Line
+	1550 3350 1950 3350
+Connection ~ 1950 3350
+Wire Wire Line
+	1950 3350 2150 3350
+$Comp
+L power:GND #PWR?
+U 1 1 606DCA08
+P 2450 3850
+F 0 "#PWR?" H 2450 3600 50  0001 C CNN
+F 1 "GND" H 2455 3677 50  0000 C CNN
+F 2 "" H 2450 3850 50  0001 C CNN
+F 3 "" H 2450 3850 50  0001 C CNN
+	1    2450 3850
+	1    0    0    -1
+$EndComp
+Wire Wire Line
+	2450 3550 2450 3850
 $EndSCHEMATC

Commit message: DOORSENSOR 9V KiCAD added
Parts:
- C1: value CP -> 220uF
- C2: value C -> 100nF
- R1: value R -> 22k
Changed lines of the file:
@@
 P 1550 3600
 F 0 "C1" H 1668 3646 50  0000 L CNN
-F 1 "CP" H 1668 3555 50  0000 L CNN
+F 1 "220uF" H 1668 3555 50  0000 L CNN
 F 2 "Capacitor_THT:CP_Radial_D6.3mm_P2.50mm" H 1588 3450 50  0001 C CNN
 F 3 "~" H 1550 3600 50  0001 C CNN
@@
 P 1950 3600
 F 0 "R1" H 2020 3646 50  0000 L CNN
-F 1 "R" H 2020 3555 50  0000 L CNN
+F 1 "22k" H 2020 3555 50  0000 L CNN
 F 2 "Resistor_THT:R_Axial_DIN0207_L6.3mm_D2.5mm_P10.16mm_Horizontal" V 1880 3600 50  0001 C CNN
 F 3 "~" H 1950 3600 50  0001 C CNN
@@
 P 3550 3250
 F 0 "C2" V 3298 3250 50  0000 C CNN
-F 1 "C" V 3389 3250 50  0000 C CNN
+F 1 "100nF" V 3389 3250 50  0000 C CNN
 F 2 "Capacitor_SMD:C_1206_3216Metric_Pad1.33x1.80mm_HandSolder" H 3588 3100 50  0001 C CNN
 F 3 "~" H 3550 3250 50  0001 C CNN
