File: KiCAD/IM350_AM550_5V_V2.0/IM350_AM550_5V_V2.0.kicad_pcb (KiCad board)
At the start: 2 copper layers, 42 x 19 mm, 10 parts, among them J5 USB_B_Micro_Power, J7 RJ12, P3 0R, P4 0R, SW1 Pairing, U1 MCP1700-3302E_SOT23, U2 ESP-12F

Commit message: Update
Parts:
- added G1: LOGO, SHRDZM:SHRDZM Symbol 5x5, F.Cu at (31.5, 40.0)
- added G2: LOGO, SHRDZM:SHRDZM 33x11, B.Cu at (51.0, 31.5)
- J7: footprint ErichCollection:RJ12_Amphenol_54601_Reduced -> Connector_PinHeader_2.54mm:PinHeader_2x03_P2.54mm_Vertical
- moved J7 2.55 mm to (30.0, 29.0), turned to 0 degrees
Routing:
- net Net-(J7-Pad2): track 20.7 -> 17.0 mm
- net Net-(J7-Pad5): track 36.9 -> 40.3 mm
- net Net-(C2-Pad2): track 72.8 -> 76.1 mm, vias 0 -> 1
- net +3V3: track 33.7 -> 32.1 mm
- net Net-(U2-Pad1): track 11.1 -> 9.92 mm
- net Net-(SW1-Pad1): track 7.58 -> 7.81 mm, vias 0 -> 2
- net Net-(J7-Pad1): track 41.7 -> 41.5 mm, vias 2 -> 1
Other:
- board text added: "V2.0"
- board text added: "www.shrdzm.com"
