File: KiCAD/IM350_AM550_5V_V2.0/IM350_AM550_5V_V2.0.sch (KiCad schematic (older format))
At the start: 10 parts, among them J5 USB_B_Micro_Power, J7 RJ12, P3 0R, P4 0R, SW1 Pairing, U1 MCP1700-3302E_SOT23, U2 ESP-12F

Commit message: Update
Parts:
- J7: footprint ErichCollection:RJ12_Amphenol_54601_Reduced -> Connector_PinHeader_2.54mm:PinHeader_2x03_P2.54mm_Vertical
Changed lines of the file:
@@
 F 0 "J7" H 8720 2404 50  0000 R CNN
 F 1 "RJ12" H 8720 2495 50  0000 R CNN
-F 2 "ErichCollection:RJ12_Amphenol_54601_Reduced" V 9050 2425 50  0001 C CNN
+F 2 "Connector_PinHeader_2.54mm:PinHeader_2x03_P2.54mm_Vertical" V 9050 2425 50  0001 C CNN
 F 3 "~" V 9050 2425 50  0001 C CNN
 	1    9050 2400
