File: KiCAD/DOORSENSOR_Simple_9V/DOORSENSOR_Simple_9V.kicad_pcb (KiCad board)
At the start: 2 copper layers, 100 x 100 mm, 130 parts, among them J1 9V, Q1 NTR4003NT1G, SW1 Trigger, SW2 Open/Close, SW3 Pairing, U1 AMS1117-3.3, U2 ESP-12F

Commit message: Update
Connections:
- R2 pad 2: GND -> Net-(Q1-Pad3) (x10)
- SW2 pad 2: GND -> Net-(Q1-Pad3) (x10)
- SW3 pad 2: GND -> Net-(Q1-Pad3) (x10)
- U2 pad 15: GND -> Net-(Q1-Pad3) (x10)
Routing:
- net Net-(Q1-Pad3): track 55.7 -> 468.7 mm, vias 0 -> 10
- net GND: track 665.0 -> 371.2 mm
- net Net-(C1-Pad1): track 284.5 -> 242.1 mm
- net +3V3: track 443.7 -> 405.2 mm
Other:
- board text added: "V1.1"
- board text removed: "V1.0"

Commit message: Update
Parts:
- removed the C1 at (55.5, 124.5)
- removed the C1 at (105.5, 124.5)
- removed the C1 at (55.5, 104.5)
- removed the C1 at (105.5, 104.5)
- removed the C1 at (105.5, 84.5)
- removed the C1 at (55.5, 84.5)
- removed the C1 at (105.5, 64.5)
- removed the C1 at (55.5, 64.5)
- removed the C1 at (105.5, 44.5)
- added C1: 100uF, Capacitor_THT:CP_Radial_D5.0mm_P2.50mm, F.Cu at (105.5, 126.5)
- added C1: 100uF, Capacitor_THT:CP_Radial_D5.0mm_P2.50mm, F.Cu at (55.5, 126.5)
- added C1: 100uF, Capacitor_THT:CP_Radial_D5.0mm_P2.50mm, F.Cu at (105.5, 106.5)
- added C1: 100uF, Capacitor_THT:CP_Radial_D5.0mm_P2.50mm, F.Cu at (55.5, 106.5)
- added C1: 100uF, Capacitor_THT:CP_Radial_D5.0mm_P2.50mm, F.Cu at (105.5, 86.5)
- added C1: 100uF, Capacitor_THT:CP_Radial_D5.0mm_P2.50mm, F.Cu at (55.5, 86.5)
- added C1: 100uF, Capacitor_THT:CP_Radial_D5.0mm_P2.50mm, F.Cu at (105.5, 66.5)
- added C1: 100uF, Capacitor_THT:CP_Radial_D5.0mm_P2.50mm, F.Cu at (55.5, 66.5)
- added C1: 100uF, Capacitor_THT:CP_Radial_D5.0mm_P2.50mm, F.Cu at (105.5, 46.5)
- added R3: 1k8, Resistor_SMD:R_0805_2012Metric_Pad1.20x1.40mm_HandSolder, F.Cu at (105.0, 121.0)
- added R3: 1k8, Resistor_SMD:R_0805_2012Metric_Pad1.20x1.40mm_HandSolder, F.Cu at (55.0, 41.0)
- added R3: 1k8, Resistor_SMD:R_0805_2012Metric_Pad1.20x1.40mm_HandSolder, F.Cu at (55.0, 121.0)
- added R3: 1k8, Resistor_SMD:R_0805_2012Metric_Pad1.20x1.40mm_HandSolder, F.Cu at (55.0, 101.0)
- added R3: 1k8, Resistor_SMD:R_0805_2012Metric_Pad1.20x1.40mm_HandSolder, F.Cu at (105.0, 101.0)
- added R3: 1k8, Resistor_SMD:R_0805_2012Metric_Pad1.20x1.40mm_HandSolder, F.Cu at (55.0, 81.0)
- added R3: 1k8, Resistor_SMD:R_0805_2012Metric_Pad1.20x1.40mm_HandSolder, F.Cu at (105.0, 81.0)
- added R3: 1k8, Resistor_SMD:R_0805_2012Metric_Pad1.20x1.40mm_HandSolder, F.Cu at (55.0, 61.0)
- added R3: 1k8, Resistor_SMD:R_0805_2012Metric_Pad1.20x1.40mm_HandSolder, F.Cu at (105.0, 61.0)
- added R3: 1k8, Resistor_SMD:R_0805_2012Metric_Pad1.20x1.40mm_HandSolder, F.Cu at (105.0, 41.0)
- moved C1 2.00 mm to (55.5, 46.5)
Connections:
- SW1 pad 2: Net-(C1-Pad1) -> Net-(R3-Pad1) (x10)
Routing:
- net Net-(C1-Pad1): track 242.1 -> 277.3 mm
- net Net-(R3-Pad1): track 0.00 -> 27.1 mm
- net GND: track 371.2 -> 349.6 mm
- net Net-(SW3-Pad1): track 199.4 -> 187.1 mm
- net Net-(U2-Pad1): track 91.5 -> 98.6 mm
- net +3V3: track 405.2 -> 400.4 mm, vias 10 -> 20
- net Net-(Q1-Pad3): track 468.7 -> 466.1 mm
- net Net-(SW2-Pad1): track 230.7 -> 232.0 mm, vias 0 -> 10
- net Net-(R2-Pad1): track 47.1 -> 48.3 mm
Other:
- board text added: "V2.0"
- board text removed: "V1.1"
