File: KiCAD/DOORSENSOR_Simple_9V/DOORSENSOR_Simple_9V_single.kicad_pcb (KiCad board)
At the start: 2 copper layers, 13 parts, among them J1 9V, Q1 NTR4003NT1G, SW1 Trigger, SW2 Open/Close, SW3 Pairing, U1 AMS1117-3.3, U2 ESP-12F

Commit message: Update
Other:
- board outline added: 50 x 20 mm

Commit message: Update
Connections:
- R2 pad 2: GND -> Net-(Q1-Pad3)
- SW2 pad 2: GND -> Net-(Q1-Pad3)
- SW3 pad 2: GND -> Net-(Q1-Pad3)
- U2 pad 15: GND -> Net-(Q1-Pad3)
Routing:
- net Net-(Q1-Pad3): track 5.57 -> 46.9 mm, vias 0 -> 1
- net GND: track 66.5 -> 37.1 mm
- net Net-(C1-Pad1): track 28.5 -> 24.2 mm
- net +3V3: track 44.4 -> 40.5 mm

Commit message: Update
Other:
- board text added: "V1.1"
- board text removed: "V1.0"

Commit message: Update
Parts:
- added R3: 1k8, Resistor_SMD:R_0805_2012Metric_Pad1.20x1.40mm_HandSolder, F.Cu at (55.0, 41.0)
- moved C1 2.00 mm to (55.5, 46.5)
Connections:
- SW1 pad 2: Net-(C1-Pad1) -> Net-(R3-Pad1)
Routing:
- net Net-(C1-Pad1): track 24.2 -> 27.7 mm
- net Net-(R3-Pad1): track 0.00 -> 2.71 mm
- net GND: track 37.1 -> 35.0 mm
- net Net-(SW3-Pad1): track 19.9 -> 18.7 mm
- net Net-(U2-Pad1): track 9.15 -> 9.86 mm
- net +3V3: track 40.5 -> 40.0 mm, vias 1 -> 2
- net Net-(SW2-Pad1): track 23.1 -> 23.2 mm, vias 0 -> 1
Other:
- board outline removed
- board text added: "V2.0"
- board text removed: "V1.1"
