File: KiCAD/IM350_AM550_T210_5V_V5.0/IM350_AM550_T210_5V_V5.0.sch (KiCad schematic (older format))
At the start: 32 parts, among them J1 USB_B_Micro_Power, J2 RJ12, Q1 BC847, SW1 SW_Push, U1 AMS1117-3.3, U2 ESP-12F, U3 TSS721ADR, U4 EL357NC, U5 EL357NC

Commit message: Update
Parts:
- U3: symbol TSS721ADR:TSS721ADR -> IM350_AM550_T210_5V_V5.0-rescue:TSS721ADR-TSS721ADR
Changed lines of the file:
@@
 NoConn ~ 1150 5400
 $Comp
-L TSS721ADR:TSS721ADR U3
+L IM350_AM550_T210_5V_V5.0-rescue:TSS721ADR-TSS721ADR U3
 U 1 1 61633360
 P 8200 2350

Commit message: MBus for Smartmeter added
Parts:
- C3: value 0.1uF -> 100nF
- C5: value 0.22uF -> 220nF
- R14: value 100k -> 100
- R16: value 10k -> 1.5k
Changed lines of the file:
@@
 U 1 1 616AFA1A
 P 10150 2350
-F 0 "R13" V 10100 2500 50  0000 C CNN
+F 0 "R13" V 10250 2350 50  0000 C CNN
 F 1 "0" V 10150 2350 50  0000 C CNN
 F 2 "Resistor_SMD:R_0201_0603Metric_Pad0.64x0.40mm_HandSolder" V 10080 2350 50  0001 C CNN
@@
 U 1 1 616F3319
 P 9350 1850
-F 0 "R11" V 9300 2000 50  0000 C CNN
+F 0 "R11" V 9450 1850 50  0000 C CNN
 F 1 "220" V 9350 1850 50  0000 C CNN
 F 2 "Resistor_SMD:R_0805_2012Metric_Pad1.20x1.40mm_HandSolder" V 9280 1850 50  0001 C CNN
@@
 U 1 1 616F3954
 P 9350 1950
-F 0 "R12" V 9300 2100 50  0000 C CNN
+F 0 "R12" V 9250 1950 50  0000 C CNN
 F 1 "220" V 9350 1950 50  0000 C CNN
 F 2 "Resistor_SMD:R_0805_2012Metric_Pad1.20x1.40mm_HandSolder" V 9280 1950 50  0001 C CNN
@@
 P 6900 2400
 F 0 "C3" H 7015 2446 50  0000 L CNN
-F 1 "0.1uF" H 7015 2355 50  0000 L CNN
+F 1 "100nF" H 7015 2355 50  0000 L CNN
 F 2 "Capacitor_SMD:C_1206_3216Metric_Pad1.33x1.80mm_HandSolder" H 6938 2250 50  0001 C CNN
 F 3 "~" H 6900 2400 50  0001 C CNN
@@
 U 1 1 616FAFE9
 P 6500 2400
-F 0 "R4" V 6450 2550 50  0000 C CNN
+F 0 "R4" V 6400 2400 50  0000 C CNN
 F 1 "100k" V 6500 2400 50  0000 C CNN
 F 2 "Resistor_SMD:R_0805_2012Metric_Pad1.20x1.40mm_HandSolder" V 6430 2400 50  0001 C CNN
@@
 U 1 1 616FEF63
 P 9600 2700
-F 0 "R14" V 9550 2850 50  0000 C CNN
-F 1 "100k" V 9600 2700 50  0000 C CNN
+F 0 "R14" V 9700 2700 50  0000 C CNN
+F 1 "100" V 9600 2700 50  0000 C CNN
 F 2 "Resistor_SMD:R_0805_2012Metric_Pad1.20x1.40mm_HandSolder" V 9530 2700 50  0001 C CNN
 F 3 "~" H 9600 2700 50  0001 C CNN
@@
 U 1 1 6173F40B
 P 9750 2700
-F 0 "R15" V 9700 2850 50  0000 C CNN
+F 0 "R15" V 9850 2700 50  0000 C CNN
 F 1 "30k" V 9750 2700 50  0000 C CNN
 F 2 "Resistor_SMD:R_0805_2012Metric_Pad1.20x1.40mm_HandSolder" V 9680 2700 50  0001 C CNN
@@
 U 1 1 61763C16
 P 9350 2900
-F 0 "C5" H 9465 2946 50  0000 L CNN
-F 1 "0.22uF" H 9465 2855 50  0000 L CNN
+F 0 "C5" H 9150 2950 50  0000 L CNN
+F 1 "220nF" H 9350 2800 50  0000 L CNN
 F 2 "Capacitor_SMD:C_1206_3216Metric_Pad1.33x1.80mm_HandSolder" H 9388 2750 50  0001 C CNN
 F 3 "~" H 9350 2900 50  0001 C CNN
@@
 U 1 1 61789B8F
 P 6150 2000
-F 0 "R17" V 6100 2150 50  0000 C CNN
+F 0 "R17" V 6050 2000 50  0000 C CNN
 F 1 "10k" V 6150 2000 50  0000 C CNN
 F 2 "Resistor_SMD:R_0805_2012Metric_Pad1.20x1.40mm_HandSolder" V 6080 2000 50  0001 C CNN
@@
 U 1 1 61790C22
 P 4550 950
-F 0 "R16" V 4500 1100 50  0000 C CNN
-F 1 "10k" V 4550 950 50  0000 C CNN
+F 0 "R16" V 4450 950 50  0000 C CNN
+F 1 "1.5k" V 4550 950 50  0000 C CNN
 F 2 "Resistor_SMD:R_0805_2012Metric_Pad1.20x1.40mm_HandSolder" V 4480 950 50  0001 C CNN
 F 3 "~" H 4550 950 50  0001 C CNN
